Commit message: 终于跑通啦！！！

File: legged_gym/resources/robots/fall_arm/fall_arm.urdf (robot description, URDF)
Before this commit: robot fall_arm, 7 links, 6 joints
Joints:
- joint left_shoulder_root_joint: limit lower=0 upper=1 effort=0 velocity=0 -> lower=0 upper=1 effort=120 velocity=20

Commit message: 1

File: legged_gym/resources/robots/fall_arm/fall_arm.urdf (robot description, URDF)
Before this commit: robot fall_arm, 7 links, 6 joints
Joints:
- joint left_shoulder_pitch_joint: origin xyz=0 0.0930000000000007 0 rpy=0 0 0 -> xyz=0 0.093 0 rpy=0 0 0

Commit message: base不可碰撞

File: legged_gym/resources/robots/fall_arm/fall_arm.urdf (robot description, URDF)
Before this commit: robot fall_arm, 7 links, 6 joints
Links:
- link base_framework: geometry visual mesh filename=meshes/base_framework.stl

Commit message: 1

File: legged_gym/resources/robots/fall_arm/fall_arm.urdf (robot description, URDF)
Before this commit: robot fall_arm, 7 links, 6 joints
Links:
- link base_framework: geometry collision mesh filename=meshes/base_framework.stl; visual mesh filename=meshes/base_framework.stl
- link end_effector: mass 0.008061 -> 0.026024
Joints:
- joint left_shoulder_pitch_joint: origin xyz=0 0.093 0 rpy=0 0 0 -> xyz=0 0.0930000000000007 0 rpy=0 0 0

Commit message: 1

File: legged_gym/resources/robots/fall_arm/fall_arm.urdf (robot description, URDF)
Before this commit: robot fall_arm, 7 links, 6 joints
Links:
- link base_framework: geometry visual mesh filename=meshes/base_framework.stl
- link end_effector: mass 0.026024 -> 0.025241

Commit message: 1

File: legged_gym/resources/robots/fall_arm/fall_arm.urdf (robot description, URDF)
Before this commit: robot fall_arm, 7 links, 6 joints
Links:
- link end_effector: mass 0.025241 -> 0.026024

Commit message: 1

File: legged_gym/resources/robots/fall_arm/fall_arm.urdf (robot description, URDF)
Before this commit: robot fall_arm, 7 links, 6 joints
Links:
- link end_effector: mass 0.026024 -> 0.025241

Commit message: 1

File: legged_gym/resources/robots/fall_arm/fall_arm.urdf (robot description, URDF)
Before this commit: robot fall_arm, 7 links, 6 joints
Joints:
- joint left_elbow_joint: limit lower=0.17453292519943295 upper=2.007128639793479 effort=120 velocity=20 -> lower=0.17453292519943295 upper=2.007128639793479 effort=144 velocity=20
- joint left_shoulder_pitch_joint: limit lower=-1.5707963267948966 upper=1.5707963267948966 effort=120 velocity=20 -> lower=-1.5707963267948966 upper=1.5707963267948966 effort=144 velocity=20
- joint left_shoulder_roll_joint: limit lower=-0.17453292519943295 upper=1.5707963267948966 effort=120 velocity=20 -> lower=-0.17453292519943295 upper=1.5707963267948966 effort=144 velocity=20
- joint left_shoulder_root_joint: limit lower=0 upper=1 effort=120 velocity=20 -> lower=0 upper=1 effort=144 velocity=20
- joint left_shoulder_yaw_joint: limit lower=-1.5707963267948966 upper=0.7853981633974483 effort=120 velocity=20 -> lower=-1.5707963267948966 upper=0.7853981633974483 effort=144 velocity=20

Commit message: 可行

File: legged_gym/resources/robots/fall_arm/fall_arm.urdf (robot description, URDF)
Before this commit: robot fall_arm, 7 links, 6 joints
Joints:
- joint left_elbow_joint: limit lower=0.17453292519943295 upper=2.007128639793479 effort=144 velocity=20 -> lower=-1.1397000015522971 upper=0.6928957130417489 effort=144 velocity=20; origin xyz=0 0 -0.261 rpy=0 0 0 -> xyz=0 0 -0.261 rpy=0 -1.314 0

Commit message: 可行

File: legged_gym/resources/robots/fall_arm/fall_arm.urdf (robot description, URDF)
Before this commit: robot fall_arm, 7 links, 6 joints
Joints:
- joint left_elbow_joint: limit lower=-1.1397000015522971 upper=0.6928957130417489 effort=144 velocity=20 -> lower=0.17453292519943295 upper=2.007128639793479 effort=144 velocity=20; origin xyz=0 0 -0.261 rpy=0 -1.314 0 -> xyz=0 0 -0.261 rpy=0 0 0
- joint left_shoulder_pitch_joint: limit lower=-1.5707963267948966 upper=1.5707963267948966 effort=144 velocity=20 -> lower=0.0 upper=1.5707963267948966 effort=144 velocity=20
- joint left_shoulder_roll_joint: limit lower=-0.17453292519943295 upper=1.5707963267948966 effort=144 velocity=20 -> lower=-0.17453292519943295 upper=0.17453292519943295 effort=144 velocity=20
- joint left_shoulder_yaw_joint: limit lower=-1.5707963267948966 upper=0.7853981633974483 effort=144 velocity=20 -> lower=-0.17453292519943295 upper=0.17453292519943295 effort=144 velocity=20

Commit message: 1

File: legged_gym/resources/robots/fall_arm/fall_arm.urdf (robot description, URDF)
Before this commit: robot fall_arm, 7 links, 6 joints
Joints:
- joint left_elbow_joint: limit lower=0.17453292519943295 upper=2.007128639793479 effort=144 velocity=20 -> lower=0.17453292519943295 upper=2.007128639793479 effort=173 velocity=20
